Commit message: [fix]修改Opendog文件使用

File: resources/robots/Opendoge/urdf/Opendoge.urdf (robot description, URDF)
Before this commit: robot Opendoge, 17 links, 16 joints
Joints:
- joint FL_calf_joint: limit lower=-2.68 upper=-1.04 effort=0 velocity=0 -> lower=-2.68 upper=-1.04 effort=9 velocity=6.981
- joint FL_hip_joint: limit lower=-0.785 upper=0.26 effort=0 velocity=0 -> lower=-0.785 upper=0.26 effort=6 velocity=10.472
- joint FL_thigh_joint: limit lower=-0.785 upper=0.785 effort=0 velocity=0 -> lower=-0.785 upper=0.785 effort=6 velocity=10.472
- joint FR_calf_joint: limit lower=-2.68 upper=-1.04 effort=0 velocity=0 -> lower=-2.68 upper=-1.04 effort=9 velocity=6.981
- joint FR_hip_joint: limit lower=-0.26 upper=0.785 effort=0 velocity=0 -> lower=-0.26 upper=0.785 effort=6 velocity=10.472
- joint FR_thigh_joint: limit lower=-0.785 upper=0.785 effort=0 velocity=0 -> lower=-0.785 upper=0.785 effort=6 velocity=10.472
- joint RL_calf_joint: limit lower=-2.68 upper=-1.04 effort=0 velocity=0 -> lower=-2.68 upper=-1.04 effort=9 velocity=6.981
- joint RL_hip_joint: limit lower=-0.785 upper=0.26 effort=0 velocity=0 -> lower=-0.785 upper=0.26 effort=6 velocity=10.472
- joint RL_thigh_joint: limit lower=-0.785 upper=0.785 effort=0 velocity=0 -> lower=-0.785 upper=0.785 effort=6 velocity=10.472
- joint RR_calf_joint: limit lower=-2.68 upper=-1.04 effort=0 velocity=0 -> lower=-2.68 upper=-1.04 effort=9 velocity=6.981
- joint RR_hip_joint: limit lower=-0.26 upper=0.785 effort=0 velocity=0 -> lower=-0.26 upper=0.785 effort=6 velocity=10.472
- joint RR_thigh_joint: limit lower=-0.785 upper=0.785 effort=0 velocity=0 -> lower=-0.785 upper=0.785 effort=6 velocity=10.472
